File: projects/Mouse Backpack/scheme.sch (EAGLE design)
At the start: 56 parts, among them J1 USB MICRO, Q1 BSS138, Q2 BSS138, U3 ATMEGA32U4-XUMU, U4 NRF8001, X1 16MHz, X2 32.768kHz, Y1 16MHz KX-7

Commit message: Разводка nRF и ADXL345
Разводка nRF и ADXL345, небольшие изменения в принципиальной схеме
adxl345
Parts:
- removed Q1, Q2: BSS138, microbuilder:MOSFET-NWIDE
- removed RN1: 10K, resistor-dil:4R-NCAY16
- added R5, R6, R7: 10k, SparkFun:RESISTOR0603-RES
Connections:
- net 3.3V: now also R5.2, R6.2, R7.2; no longer Q1.G, Q2.G, RN1A.2, RN1B.2, RN4B.2
- net CS: now also R5.1; no longer RN4B.1
- net SCL: now also R7.1; no longer Q2.S, RN1B.1
- net SCL_5V: no longer Q2.D, RN1D.1
- net SDA/SDIO: now also R6.1; no longer Q1.S, RN1A.1
- net SDA/SDIO_5V: no longer Q1.D, RN1C.1
- net VIN: no longer RN1C.2, RN1D.2
Changed lines of the file:
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@@
 <part name="C9" library="adafruit" deviceset="C-US" device="C0805" value="10µF"/>
 <part name="U$15" library="microbuilder" deviceset="GND" device=""/>
-<part name="Q1" library="microbuilder" deviceset="MOSFET-N" device="WIDE" value="BSS138"/>
-<part name="Q2" library="microbuilder" deviceset="MOSFET-N" device="WIDE" value="BSS138"/>
-<part name="U$16" library="microbuilder" deviceset="VIN" device=""/>
-<part name="U$17" library="microbuilder" deviceset="VIN" device=""/>
 <part name="U1" library="microbuilder" deviceset="ACCEL_ADXL345" device=""/>
 <part name="ICSP" library="SmartPrj" deviceset="PINHD-2X3" device="" value="ICSP"/>
@@
 <part name="GND23" library="supply1" deviceset="GND" device=""/>
 <part name="RN4" library="resistor-dil" deviceset="4R-N" device="CAY16" value="10K"/>
-<part name="RN1" library="resistor-dil" deviceset="4R-N" device="CAY16" value="10K"/>
 <part name="U4" library="FitnessDevice" deviceset="NRF8001" device=""/>
 <part name="C2" library="SparkFun" deviceset="CAP" device="0603-CAP" value="100nF"/>
@@
 <part name="U$3" library="ant-planar-1" deviceset="ANTENNA_1" device="LEFT"/>
 <part name="VIN8" library="microbuilder" deviceset="VIN" device=""/>
+<part name="R5" library="SparkFun" deviceset="RESISTOR" device="0603-RES" value="10k"/>
+<part name="R6" library="SparkFun" deviceset="RESISTOR" device="0603-RES" value="10k"/>
+<part name="R7" library="SparkFun" deviceset="RESISTOR" device="0603-RES" value="10k"/>
 </parts>
 <sheets>
@@
 <instance part="C9" gate="G$1" x="281.94" y="2.54"/>
 <instance part="U$15" gate="G$1" x="281.94" y="-10.16"/>
-<instance part="Q1" gate="G$1" x="251.46" y="35.56" rot="R270"/>
-<instance part="Q2" gate="G$1" x="261.62" y="25.4" rot="R270"/>
-<instance part="U$16" gate="G$1" x="264.16" y="50.8"/>
-<instance part="U$17" gate="G$1" x="271.78" y="50.8"/>
 <instance part="U1" gate="G$1" x="231.14" y="-25.4"/>
 <instance part="ICSP" gate="A" x="7.62" y="73.66" smashed="yes">
@@
 <instance part="GND23" gate="1" x="142.24" y="0" rot="R90"/>
 <instance part="RN4" gate="A" x="71.12" y="58.42" rot="R90"/>
-<instance part="RN4" gate="B" x="264.16" y="-7.62" rot="R90"/>
 <instance part="RN4" gate="C" x="129.54" y="0" rot="R180"/>
 <instance part="RN4" gate="D" x="0" y="38.1" rot="R90"/>
-<instance part="RN1" gate="A" x="233.68" y="40.64" rot="R90"/>
-<instance part="RN1" gate="B" x="241.3" y="40.64" rot="R90"/>
-<instance part="RN1" gate="C" x="264.16" y="40.64" rot="R90"/>
-<instance part="RN1" gate="D" x="271.78" y="40.64" rot="R90"/>
 <instance part="U4" gate="G$1" x="302.26" y="-134.62"/>
 <instance part="C2" gate="G$1" x="208.28" y="-142.24"/>
@@
 <instance part="U$3" gate="G$1" x="396.24" y="-111.76" rot="MR0"/>
 <instance part="VIN8" gate="G$1" x="144.78" y="-73.66"/>
+<instance part="R5" gate="G$1" x="264.16" y="-7.62" rot="R90"/>
+<instance part="R6" gate="G$1" x="233.68" y="40.64" rot="R90"/>
+<instance part="R7" gate="G$1" x="241.3" y="40.64" rot="R90"/>
 </instances>
 <busses>
@@
 <wire x1="264.16" y1="-15.24" x2="264.16" y2="-12.7" width="0.1524" layer="91"/>
 <pinref part="U1" gate="G$1" pin="CS"/>
-<pinref part="RN4" gate="B" pin="1"/>
+<pinref part="R5" gate="G$1" pin="1"/>
 </segment>
 </net>
@@
 </segment>
 <segment>
-<pinref part="Q2" gate="G$1" pin="S"/>
 <wire x1="256.54" y1="22.86" x2="241.3" y2="22.86" width="0.1524" layer="91"/>
 <label x="218.44" y="22.86" size="1.778" layer="95"/>
@@
 <wire x1="241.3" y1="35.56" x2="241.3" y2="22.86" width="0.1524" layer="91"/>
 <junction x="241.3" y="22.86"/>
-<pinref part="RN1" gate="B" pin="1"/>
+<pinref part="R7" gate="G$1" pin="1"/>
 </segment>
 </net>
@@
 </segment>
 <segment>
-<pinref part="Q1" gate="G$1" pin="S"/>
 <wire x1="246.38" y1="33.02" x2="233.68" y2="33.02" width="0.1524" layer="91"/>
 <label x="218.44" y="33.02" size="1.778" layer="95"/>
@@
 <wire x1="233.68" y1="35.56" x2="233.68" y2="33.02" width="0.1524" layer="91"/>
 <junction x="233.68" y="33.02"/>
-<pinref part="RN1" gate="A" pin="1"/>
+<pinref part="R6" gate="G$1" pin="1"/>
 </segment>
 </net>
@@
 <pinref part="U$10" gate="G$1" pin="3.3V"/>
 <wire x1="233.68" y1="45.72" x2="233.68" y2="48.26" width="0.1524" layer="91"/>
-<pinref part="RN1" gate="A" pin="2"/>
+<pinref part="R6" gate="G$1" pin="2"/>
 </segment>
 <segment>
 <pinref part="U$11" gate="G$1" pin="3.3V"/>
 <wire x1="241.3" y1="45.72" x2="241.3" y2="48.26" width="0.1524" layer="91"/>
-<pinref part="Q1" gate="G$1" pin="G"/>
-<wire x1="248.92" y1="38.1" x2="248.92" y2="48.26" width="0.1524" layer="91"/>
-<wire x1="248.92" y1="48.26" x2="241.3" y2="48.26" width="0.1524" layer="91"/>
-<junction x="241.3" y="48.26"/>
-<pinref part="Q2" gate="G$1" pin="G"/>
-<wire x1="259.08" y1="27.94" x2="259.08" y2="48.26" width="0.1524" layer="91"/>
-<wire x1="259.08" y1="48.26" x2="248.92" y2="48.26" width="0.1524" layer="91"/>
-<junction x="248.92" y="48.26"/>
-<pinref part="RN1" gate="B" pin="2"/>
+<pinref part="R7" gate="G$1" pin="2"/>
 </segment>
 <segment>
@@
 <segment>
 <pinref part="U$12" gate="G$1" pin="3.3V"/>
-<pinref part="RN4" gate="B" pin="2"/>
+<pinref part="R5" gate="G$1" pin="2"/>
 </segment>
 </net>
@@
 <wire x1="281.94" y1="7.62" x2="281.94" y2="5.08" width="0.1524" layer="91"/>
 <junction x="281.94" y="7.62"/>
-</segment>
-<segment>
-<pinref part="U$16" gate="G$1" pin="VIN"/>
-<wire x1="264.16" y1="48.26" x2="264.16" y2="45.72" width="0.1524" layer="91"/>
-<pinref part="RN1" gate="C" pin="2"/>
-</segment>
-<segment>
-<pinref part="U$17" gate="G$1" pin="VIN"/>
-<wire x1="271.78" y1="48.26" x2="271.78" y2="45.72" width="0.1524" layer="91"/>
-<pinref part="RN1" gate="D" pin="2"/>
 </segment>
 <segment>
@@
 <net name="SDA/SDIO_5V" class="0">
 <segment>
-<pinref part="Q1" gate="G$1" pin="D"/>
-<wire x1="256.54" y1="33.02" x2="264.16" y2="33.02" width="0.1524" layer="91"/>
-<wire x1="264.16" y1="33.02" x2="294.64" y2="33.02" width="0.1524" layer="91"/>
-<wire x1="264.16" y1="35.56" x2="264.16" y2="33.02" width="0.1524" layer="91"/>
-<junction x="264.16" y="33.02"/>
-<label x="276.86" y="33.02" size="1.778" layer="95"/>
-<pinref part="RN1" gate="C" pin="1"/>
-</segment>
-<segment>
 <wire x1="119.38" y1="-43.18" x2="137.16" y2="-43.18" width="0.1524" layer="91"/>
 <label x="129.54" y="-43.18" size="1.778" layer="95"/>
@@
 <net name="SCL_5V" class="0">
 <segment>
-<pinref part="Q2" gate="G$1" pin="D"/>
-<wire x1="266.7" y1="22.86" x2="271.78" y2="22.86" width="0.1524" layer="91"/>
-<wire x1="271.78" y1="22.86" x2="294.64" y2="22.86" width="0.1524" layer="91"/>
-<wire x1="271.78" y1="35.56" x2="271.78" y2="22.86" width="0.1524" layer="91"/>
-<junction x="271.78" y="22.86"/>
-<label x="284.48" y="22.86" size="1.778" layer="95"/>
-<pinref part="RN1" gate="D" pin="1"/>
-</segment>
-<segment>
 <wire x1="119.38" y1="-45.72" x2="137.16" y2="-45.72" width="0.1524" layer="91"/>
